File: projects/nixie-clock/nixie-clock.sch (EAGLE design)
At the start: 33 parts, among them IC1 REG1117, T1 BC337, U1 ARDUINO_PRO_MINI_TS, U2 K155ID1, U3 CHINA_HV_DC_DC, U4 DCF1

Commit message: Update nixie-clock
Parts:
- removed C2: 100uF/25v, rcl:CPOL-EUE2.5-6
- added C10, C12: 220nF, rcl:C-EU025-024X044
- added C11: 470nF, rcl:C-EU025-024X044
- added C9: 100uF/25V, rcl:CPOL-EUE2.5-6
- added D4, D5: 1N4004, diode:1N4004
- added J1: POWER_JACKSLT, SparkFun-Connectors:POWER_JACKSLT
- added L2, L3: (no value), microfarad-de:CHOKE/9.5MM
- added R2, R3, R4, R5, R6, R7, R8, R9: (no value), rcl:R-EU_0207/7
- C3: value 100uF/25v -> 100uF/25V
- C4: value 10uF/50v -> 10uF/50V
- D3: device diode:ZENER-DIODEDO35Z10 -> diode:ZENER-DIODEZD-5
- L1: value CHOKE/9.5MM -> (none); device karim:CHOKE/9.5MM -> microfarad-de:CHOKE/9.5MM
Connections:
- removed net GND: U1.GND, U2.GND
- new net +12V: C3.+, C6.1, C7.1, IC1.VIN, L1.2, L2.2
- new net +3V3: C4.+, D3.C, R1.1
- new net 0V: C10.2, C11.2, C12.2, C3.-, C4.-, C5.-, C6.2, C7.2, C9.-, D3.A, IC1.GND, J1.GND, R3.1, R7.1, R8.1, R9.1, T1.E, U1.GND, U2.GND, U3.GND, U3.GND_OUT
- new net 180V: L3.2, R2.2, R6.2
- new net 180VRAW: L3.1, U3.UH_OUT
- new net N$10: OK5.A, U1.4
- new net N$11: OK4.A, U1.7
- new net N$12: D4.A, OK3.A, U1.*10
- new net N$13: D2.A, OK2.A, U1.*11
- new net N$14: OK1.A, U1.12
- new net N$15: L1.1, R5.1, U3.U_IN
- new net N$16: R4.2, T1.B
- new net N$17: C5.+, D2.C, D4.C, R4.1
- new net N$18: R5.2, T1.C, U3.SHDN
- new net N$19: OK1.C, OK2.C, OK3.C, OK4.C, OK5.C, OK6.C, R3.2
- new net N$20: OK7.C, R7.2
- new net N$21: OK7.A, U1.TXO
- new net N$22: OK8.EMIT, R8.2
- new net N$23: OK8.C, R9.2
- new net N$24: OK8.A, U1.13
- new net N$25: D5.A, J1.PWR
- new net N$26: D5.C, L2.1
- new net N$9: OK6.A, U1.2
- net +5V: now also C10.1, C11.1, C12.1, C9.+, IC1.VOUT, R1.2
- net B10: now also OK8.COL
- net N$7: now also OK7.EMIT, R2.1
- net N$8: now also OK7.COL, R6.1; no longer OK1.C, OK2.C, OK3.C, OK4.C, OK5.C, OK6.C
Other:
- moved on the sheet: C1, C3, C4, C5, C6, C7, D1, D2, IC1, OK7, OK8, R1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

Commit message: Finalized circuit diagram
Parts:
- removed IC1: REG1117, burr-brown:REG1117
- added C13, C2, C8: 220nF, rcl:C-EU025-024X044
- added D6, D7: 1N4148, diode:1N4148DO35-7
- added R10: 33K, rcl:R-EU_0207/7
- added R11, R13: 100K, rcl:R-EU_0207/7
- added R12: 1M, rcl:R-EU_0207/7
- added R14: 10K, rcl:R-EU_0207/7
- added R15, R23, R24, R25: 56K, rcl:R-EU_0207/7
- added R16: 670K, rcl:R-EU_0207/7
- added R17: 220K, rcl:R-EU_0207/7
- added R18: Photoresistor, SparkFun-Sensors:PHOTOCELLPTH
- added R19: 67K, rcl:R-EU_0207/7
- added R20, R21, R22: 22K, rcl:R-EU_0207/7
- added S1: "Decrease", SparkFun-Switches:MOMENTARY-SWITCH-SPST-PTH-6.0MM
- added S2: "Mode", SparkFun-Switches:MOMENTARY-SWITCH-SPST-PTH-6.0MM
- added S3: "Increase", SparkFun-Switches:MOMENTARY-SWITCH-SPST-PTH-6.0MM
- added T2, T3: BC337, transistor:BC337
- added U5: REG1117, burr-brown:REG1117
- C11, C7: value 470nF -> 220nF
- C5: value 1uF/63v -> 1uF/63V
- D1: value 1N5819-B -> 1N5819
- D2: value 1N4004 -> 1N5819-B; device diode:1N4004 -> diode:1N5819-B
- D4: value 1N4004 -> 1N5819; device diode:1N4004 -> diode:1N5819-B
- J1: value POWER_JACKSLT -> POWER JACK
- L1, L2, L3: value (none) -> 10uH
- R1: value (none) -> 1K
- R2: value (none) -> 8K2
- R3, R7, R9: value (none) -> 670
- R4: value (none) -> 100K
- R5: value (none) -> 270K
- R6: value (none) -> 6K7
- R8: value (none) -> 10K
- U1: value ARDUINO_PRO_MINI_TS -> Arduino Pro Mini
- U3: value CHINA_HV_DC_DC -> DC-DC Converter
- U4: value DCF1 -> Pollin DCF1
Connections:
- new net N$27: R10.2, R12.1, T2.C, U1.*3
- new net N$28: R13.1, R14.2, T3.B
- new net N$29: R11.1, T2.B
- new net N$30: R11.2, U4.DATA
- new net N$31: SG1.1, T3.C
- new net N$32: R14.1, U1.RXI
- new net N$33: C1.+, C11.1, D1.C, R16.2, U1.VCC
- new net N$34: R16.1, R17.1, U1.A7
- new net N$35: D2.C, D4.A, R15.1, U1.A0
- new net N$36: R15.2, R18.P$2, R19.2
- new net N$37: R20.2, R23.2, S1.2
- new net N$38: R21.2, R24.2, S2.2
- new net N$39: R22.2, R25.2, S3.2
- new net N$40: R23.1, U1.A1
- new net N$41: R24.1, U1.A2
- new net N$42: R25.1, U1.A3
- net +12V: now also U5.VIN; no longer IC1.VIN
- net +3V3: now also C2.1, U4.VCC
- net +5V: now also D1.A, D4.C, R10.1, R19.1, R20.1, R21.1, R22.1, SG1.2, U1.A6, U5.VOUT; no longer C11.1, IC1.VOUT, U1.VCC
- net 0V: now also C1.-, C13.2, C2.2, C8.2, D2.A, R12.2, R13.2, R17.2, R18.P$1, S1.1, S2.1, S3.1, T2.E, T3.E, U4.GND, U4.PON, U5.GND; no longer IC1.GND
- net N$12: now also D6.A; no longer D4.A
- net N$13: now also D7.A; no longer D2.A
- net N$15: now also C13.1
- net N$17: now also D6.C, D7.C; no longer D2.C, D4.C
- net N$26: now also C8.1
Other:
- note added: "Brightness Boost"
- note added: "Buzzer"
- note added: "DCF 77 Receiver"
- note added: "Decimal Point"
- note added: "High Voltage Activation"
- note added: "High Voltage Generator"
- note added: "Power Supply"
- note added: "Supercap."
- moved on the sheet: C1, C10, C11, C3, C4, C5, C6, C7, C9, D1, D3, J1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
