File: projects/nixie-clock/nixie-clock.brd (EAGLE design)
At the start: 124.1 x 80 mm, 33 parts, among them IC1 REG1117, T1 BC337, U1 ARDUINO_PRO_MINI_TS, U2 K155ID1, U3 CHINA_HV_DC_DC, U4 DCF1

Commit message: Update nixie-clock
Parts:
- removed C2: 100uF/25v, rcl:E2,5-6
- added C10, C12: 220nF, rcl:C025-024X044
- added C11: 470nF, rcl:C025-024X044
- added C9: 100uF/25V, rcl:E2,5-6
- added D4, D5: 1N4004, diode:DO41-10
- added J1: POWER_JACKSLT, SparkFun-Connectors:POWER_JACK_SLOT
- added L2, L3: (no value), microfarad-de:CHOKE/9.5MM
- added R2, R3, R4, R5, R6, R7, R8, R9: (no value), rcl:0207/7
- C3: value 100uF/25v -> 100uF/25V
- C4: value 10uF/50v -> 10uF/50V
- D3: device diode:DO35Z10 -> diode:ZDIO-5
- L1: value CHOKE/9.5MM -> (none); device karim:CHOKE/9.5MM -> microfarad-de:CHOKE/9.5MM
- moved L1 121.8 mm to (-1.27, -68.6)
- moved D3 33.0 mm to (-3.81, -3.81)
Connections:
- removed net GND_OUT: U3.GND_OUT
- removed net U_IN: U3.U_IN
- new net +12V: C3.+, C6.1, C7.1, IC1.3, L1.2, L2.2
- new net +3V3: C4.+, D3.C, R1.1
- new net 0V: C10.2, C11.2, C12.2, C3.-, C4.-, C5.-, C6.2, C7.2, C9.-, D3.A, IC1.1, J1.GND@2, R3.1, R7.1, R8.1, R9.1, T1.1, U1.4, U2.12, U3.GND, U3.GND_OUT
- new net 180V: L3.2, R2.2, R6.2
- new net 180VRAW: L3.1, U3.UH_OUT
- new net N$10: OK5.1, U1.7
- new net N$11: OK4.1, U1.10
- new net N$12: D4.A, OK3.1, U1.13
- new net N$13: D2.A, OK2.1, U1.14
- new net N$14: OK1.1, U1.15
- new net N$15: L1.1, R5.1, U3.U_IN
- new net N$16: R4.2, T1.2
- new net N$17: C5.+, D2.C, D4.C, R4.1
- new net N$18: R5.2, T1.3, U3.SHDN
- new net N$19: OK1.2, OK2.2, OK3.2, OK4.2, OK5.2, OK6.2, R3.2
- new net N$20: OK7.2, R7.2
- new net N$21: OK7.1, U1.1
- new net N$22: OK8.3, R8.2
- new net N$23: OK8.2, R9.2
- new net N$24: OK8.1, U1.16
- new net N$25: D5.A, J1.PWR
- new net N$26: D5.C, L2.1
- new net N$9: OK6.1, U1.5
- net +5V: now also C10.1, C11.1, C12.1, C9.+, IC1.2, R1.2
- net B10: now also OK8.4
- net GND: no longer IC1.1, U1.4, U2.12, U3.GND
- net N$7: now also OK7.3, R2.1
- net N$8: now also OK7.4, R6.1; no longer OK1.2, OK2.2, OK3.2, OK4.2, OK5.2, OK6.2
Routing:
- net N$8: track 118.4 -> 0.00 mm, vias 2 -> 0
- net N$19: track 0.00 -> 118.2 mm, vias 0 -> 2
- net GND: track 47.8 -> 17.3 mm

Commit message: Finalized circuit diagram
Parts:
- added C13, C2, C8: 220nF, rcl:C025-024X044
- added D6, D7: 1N4148, diode:DO35-7
- added R10: 33K, rcl:0207/7
- added R11, R13: 100K, rcl:0207/7
- added R12: 1M, rcl:0207/7
- added R14: 10K, rcl:0207/7
- added R15, R23, R24, R25: 56K, rcl:0207/7
- added R16: 670K, rcl:0207/7
- added R17: 220K, rcl:0207/7
- added R18: Photoresistor, SparkFun-Sensors:PHOTOCELL
- added R19: 67K, rcl:0207/7
- added R20, R21, R22: 22K, rcl:0207/7
- added S1: "Decrease", SparkFun-Switches:TACTILE_SWITCH_PTH_6.0MM
- added S2: "Mode", SparkFun-Switches:TACTILE_SWITCH_PTH_6.0MM
- added S3: "Increase", SparkFun-Switches:TACTILE_SWITCH_PTH_6.0MM
- added T2, T3: BC337, transistor:TO92
- C11, C7: value 470nF -> 220nF
- C5: value 1uF/63v -> 1uF/63V
- D1: value 1N5819-B -> 1N5819
- D2: value 1N4004 -> 1N5819-B; device diode:DO41-10 -> diode:DO41-7.6
- D4: value 1N4004 -> 1N5819; device diode:DO41-10 -> diode:DO41-7.6
- J1: value POWER_JACKSLT -> POWER JACK
- L1, L2, L3: value (none) -> 10uH
- R1: value (none) -> 1K
- R2: value (none) -> 8K2
- R3, R7, R9: value (none) -> 670
- R4: value (none) -> 100K
- R5: value (none) -> 270K
- R6: value (none) -> 6K7
- R8: value (none) -> 10K
- U1: value ARDUINO_PRO_MINI_TS -> Arduino Pro Mini
- U3: value CHINA_HV_DC_DC -> DC-DC Converter
- U4: value DCF1 -> Pollin DCF1
- moved D2 330.7 mm to (-25.4, -301.0)
- moved D4 200.8 mm to (-25.4, -278.1)
- renumbered IC1 to U5
Connections:
- removed net VCC: U4.VCC
- new net N$27: R10.2, R12.1, T2.3, U1.6
- new net N$28: R13.1, R14.2, T3.2
- new net N$29: R11.1, T2.2
- new net N$30: R11.2, U4.DATA
- new net N$31: SG1.-, T3.3
- new net N$32: R14.1, U1.2
- new net N$33: C1.+, C11.1, D1.C, R16.2, U1.21
- new net N$34: R16.1, R17.1, U1.A7
- new net N$35: D2.C, D4.A, R15.1, U1.17
- new net N$36: R15.2, R18.2, R19.2
- new net N$37: R20.2, R23.2, S1.3
- new net N$38: R21.2, R24.2, S2.3
- new net N$39: R22.2, R25.2, S3.3
- new net N$40: R23.1, U1.18
- new net N$41: R24.1, U1.19
- new net N$42: R25.1, U1.20
- net +3V3: now also C2.1, U4.VCC
- net +5V: now also D1.A, D4.C, R10.1, R19.1, R20.1, R21.1, R22.1, SG1.+, U1.A6; no longer C11.1, U1.21
- net 0V: now also C1.-, C13.2, C2.2, C8.2, D2.A, R12.2, R13.2, R17.2, R18.1, S1.1, S2.1, S3.1, T2.1, T3.1, U4.GND, U4.PON
- net GND: no longer U4.GND
- net N$12: now also D6.A; no longer D4.A
- net N$13: now also D7.A; no longer D2.A
- net N$15: now also C13.1
- net N$17: now also D6.C, D7.C; no longer D2.C, D4.C
- net N$26: now also C8.1

Commit message: Renumber parts
Parts:
- C1: value 1.5F/5.5V -> 220nF; device karim:SUPERCAP/1.5F/5.5V -> rcl:C025-024X044
- C10: value 220nF -> 1.5F/5.5V; device rcl:C025-024X044 -> karim:SUPERCAP/1.5F/5.5V
- C4: value 10uF/50V -> 220nF; device rcl:E2-4 -> rcl:C025-024X044
- C5: value 1uF/63V -> 100uF/25V; device rcl:E1,8-4 -> rcl:E2,5-6
- C6: value 220nF -> 10uF/50V; device rcl:C025-024X044 -> rcl:E2-4
- C9: value 100uF/25V -> 1uF/63V; device rcl:E2,5-6 -> rcl:E1,8-4
- D1: value 1N5819 -> 1N4004; device diode:DO41-7.6 -> diode:DO41-10
- D2: value 1N5819-B -> 3.3v; device diode:DO41-7.6 -> diode:ZDIO-5
- D3: value 3.3v -> 1N5819; device diode:ZDIO-5 -> diode:DO41-7.6
- D4: value 1N5819 -> 1N4148; device diode:DO41-7.6 -> diode:DO35-7
- D5: value 1N4004 -> 1N4148; device diode:DO41-10 -> diode:DO35-7
- D6: value 1N4148 -> 1N5819; device diode:DO35-7 -> diode:DO41-7.6
- D7: value 1N4148 -> 1N5819-B; device diode:DO35-7 -> diode:DO41-7.6
- R10: value 33K -> 100K
- R11: value 100K -> 10K
- R12: value 1M -> 100K
- R13: value 100K -> 67K
- R14: value 10K -> 22K
- R15: value 56K -> 22K
- R16: value 670K -> 22K
- R17: value 220K -> Photoresistor; device rcl:0207/7 -> SparkFun-Sensors:PHOTOCELL
- R18: value Photoresistor -> 56K; device SparkFun-Sensors:PHOTOCELL -> rcl:0207/7
- R19: value 67K -> 220K
- R20: value 22K -> 33K
- R21: value 22K -> 56K
- R22: value 22K -> 100K
- R23: value 56K -> 1M
- R3: value 670 -> 6K7
- R4: value 100K -> 670
- R6: value 6K7 -> 670
- R9: value 670 -> 670K
- U1: value Arduino Pro Mini -> DC-DC Converter; device karim:ARDUINO_PRO_MINI_TS -> karim:CHINA_HV_DC_DC
- U3: value DC-DC Converter -> Arduino Pro Mini; device karim:CHINA_HV_DC_DC -> karim:ARDUINO_PRO_MINI_TS
- moved C1 300.8 mm to (-27.9, -262.9)
- moved D2 298.0 mm to (-3.81, -3.81)
- moved C7 293.7 mm to (-27.9, -270.5)
- moved C8 286.2 mm to (27.9, 17.8)
- moved C2 169.8 mm to (27.9, 24.1)
- moved D1 152.5 mm to (-12.7, -132.1)
- moved R12 147.8 mm to (-25.4, -308.6)
- moved C13 131.3 mm to (-16.5, -139.7)
- moved R23 125.0 mm to (-14.0, -161.3)
- moved D5 116.3 mm to (-25.4, -247.7)
- moved C10 99.1 mm to (53.3, 26.7)
- moved R13 87.6 mm to (-25.4, -221.0)
- moved R22 80.8 mm to (-14.0, -156.2)
- moved R20 75.8 mm to (-14.0, -151.1)
- moved C4 68.3 mm to (-5.08, -53.3)
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Connections:
- net +12V: now also C2.1, C8.1; no longer C6.1, C7.1
- net +3V3: now also C13.1, C6.+, D2.C; no longer C2.1, C4.+, D3.C
- net +5V: now also C4.1, C5.+, D3.A, D6.C, R13.1, R14.1, R15.1, R16.1, U3.A6; no longer C10.1, C9.+, D1.A, D4.C, R10.1, R19.1, R21.1, R22.1, U1.A6
- net 0V: now also C1.2, C10.-, C4.2, C6.-, D7.A, R17.1, R19.2, R23.2, R4.1, R6.1, U1.GND, U1.GND_OUT, U3.4; no longer C1.-, C10.2, C4.-, C6.2, D3.A, R13.2, R17.2, R18.1, R3.1, R9.1, U1.4, U3.GND, U3.GND_OUT
- net 180V: now also R3.2; no longer R6.2
- net 180VRAW: now also U1.UH_OUT; no longer U3.UH_OUT
- net GND: now also U3.23; no longer U1.23
- net N$10: now also U3.7; no longer U1.7
- net N$11: now also U3.10; no longer U1.10
- net N$12: now also D4.A, U3.13; no longer D6.A, U1.13
- net N$13: now also D5.A, U3.14; no longer D7.A, U1.14
- net N$14: now also U3.15; no longer U1.15
- net N$15: now also C7.1, L2.1, U1.U_IN; no longer C13.1, L1.1, U3.U_IN
- net N$16: now also R10.2; no longer R4.2
- net N$17: now also C9.+, D4.C, D5.C, R10.1; no longer C5.+, D6.C, D7.C, R4.1
- net N$18: now also U1.SHDN; no longer U3.SHDN
- net N$19: now also R4.2; no longer R3.2
- net N$20: now also R6.2; no longer R7.2
- net N$21: now also U3.1; no longer U1.1
- net N$23: now also R7.2; no longer R9.2
- net N$24: now also U3.16; no longer U1.16
- net N$25: now also D1.A; no longer D5.A
- net N$26: now also C1.1, D1.C, L1.1; no longer C8.1, D5.C, L2.1
- net N$27: now also R20.2, R23.1, T3.3, U3.6; no longer R10.2, R12.1, T2.3, U1.6
- net N$28: now also R11.2, R12.1, T2.2; no longer R13.1, R14.2, T3.2
- net N$29: now also R22.1, T3.2; no longer R11.1, T2.2
- net N$30: now also R22.2; no longer R11.2
- net N$31: now also T2.3; no longer T3.3
- net N$32: now also R11.1, U3.2; no longer R14.1, U1.2
- net N$33: now also C10.+, D3.C, R9.2, U3.21; no longer C1.+, D1.C, R16.2, U1.21
- net N$34: now also R19.1, R9.1, U3.A7; no longer R16.1, R17.1, U1.A7
- net N$35: now also D6.A, D7.C, R18.1, U3.17; no longer D2.C, D4.A, R15.1, U1.17
- net N$36: now also R13.2, R17.2; no longer R15.2, R19.2
- net N$37: now also R14.2, R21.2; no longer R20.2, R23.2
- net N$38: now also R15.2; no longer R21.2
- net N$39: now also R16.2; no longer R22.2
- net N$40: now also R21.1, U3.18; no longer R23.1, U1.18
- net N$41: now also U3.19; no longer U1.19
- net N$42: now also U3.20; no longer U1.20
- net N$8: now also R3.1; no longer R6.1
- net N$9: now also U3.5; no longer U1.5
- net RAW: now also U3.24; no longer U1.24
- net X1: now also U3.12; no longer U1.12
- net X2: now also U3.9; no longer U1.9
- net X3: now also U3.8; no longer U1.8
- net X4: now also U3.11; no longer U1.11

Commit message: Update schematic
Parts:
- removed R12: 100K, rcl:0207/7
Connections:
- net 0V: no longer R12.2
- net N$28: no longer R12.1
Changed lines of the file:
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@@
 <attribute name="VALUE" x="-27.432" y="-303.911" size="1.27" layer="27" ratio="10"/>
-</element>
-<element name="R12" library="rcl" library_urn="urn:adsk.eagle:library:334" package="0207/7" package3d_urn="urn:adsk.eagle:package:23493/2" value="100K" x="-25.4" y="-308.61" smashed="yes">
-<attribute name="NAME" x="-27.94" y="-307.213" size="1.27" layer="25" ratio="10"/>
-<attribute name="SPICEPREFIX" value="R" x="-25.4" y="-308.61" size="1.778" layer="27" display="off"/>
-<attribute name="VALUE" x="-27.686" y="-309.1688" size="1.27" layer="27" ratio="10"/>
 </element>
 </elements>
@@
 <contactref element="C7" pad="2"/>
 <contactref element="D7" pad="A"/>
-<contactref element="R12" pad="2"/>
 <wire x1="-29.9212" y1="-203.4794" x2="-29.9212" y2="-211.0994" width="0" layer="19" extent="1-1"/>
 <wire x1="-29.94" y1="-198.12" x2="-29.9212" y2="-203.4794" width="0" layer="19" extent="1-1"/>
@@
 <wire x1="-26.67" y1="-270.51" x2="-26.67" y2="-262.89" width="0" layer="19" extent="1-1"/>
 <wire x1="-21.59" y1="-300.99" x2="-26.67" y2="-270.51" width="0" layer="19" extent="1-1"/>
-<wire x1="-21.59" y1="-308.61" x2="-21.59" y2="-300.99" width="0" layer="19" extent="1-1"/>
 </signal>
 <signal name="180VRAW">
@@
 <contactref element="R11" pad="2"/>
 <contactref element="T2" pad="2"/>
-<contactref element="R12" pad="1"/>
 <wire x1="-15.24" y1="-164.465" x2="-10.16" y2="-176.53" width="0" layer="19" extent="1-1"/>
-<wire x1="-29.21" y1="-308.61" x2="-10.16" y2="-176.53" width="0" layer="19" extent="1-1"/>
 </signal>
 </signals>

Commit message: Update nixie-clock schematic
Parts:
- J1: value POWER JACK -> Power Jack
Connections:
- net 180V renamed +180V
Changed lines of the file:
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@@
 <attribute name="VALUE" x="-4.826" y="-127.5588" size="1.27" layer="27" ratio="10"/>
 </element>
-<element name="J1" library="SparkFun-Connectors" library_urn="urn:adsk.eagle:library:513" package="POWER_JACK_SLOT" package3d_urn="urn:adsk.eagle:package:38222/1" value="POWER JACK" x="-17.78" y="-127" smashed="yes">
+<element name="J1" library="SparkFun-Connectors" library_urn="urn:adsk.eagle:library:513" package="POWER_JACK_SLOT" package3d_urn="urn:adsk.eagle:package:38222/1" value="Power Jack" x="-17.78" y="-127" smashed="yes">
 <attribute name="NAME" x="-14.2748" y="-124.841" size="0.6096" layer="25" font="vector" ratio="20"/>
 <attribute name="PROD_ID" value="PRT-00119" x="-17.78" y="-127" size="1.778" layer="27" display="off"/>
@@
 <wire x1="-29.21" y1="-270.51" x2="-6.35" y2="-91.44" width="0" layer="19" extent="1-1"/>
 </signal>
-<signal name="180V">
+<signal name="+180V">
 <contactref element="L3" pad="2"/>
 <contactref element="R2" pad="2"/>

Commit message: Created schematic for the antenna tuner
Parts:
- D2: value 3.3v -> 3.3V
- D7: value 1N5819-B -> 1N5819
Changed lines of the file:
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@@
 <attribute name="VALUE" x="10.16" y="24.13" size="1.27" layer="27"/>
 </element>
-<element name="D2" library="diode" library_urn="urn:adsk.eagle:library:210" package="ZDIO-5" package3d_urn="urn:adsk.eagle:package:43412/1" value="3.3v" x="-3.81" y="-3.81" smashed="yes">
+<element name="D2" library="diode" library_urn="urn:adsk.eagle:library:210" package="ZDIO-5" package3d_urn="urn:adsk.eagle:package:43412/1" value="3.3V" x="-3.81" y="-3.81" smashed="yes">
 <attribute name="NAME" x="-6.4262" y="-1.9812" size="1.27" layer="25" ratio="10"/>
 <attribute name="VALUE" x="-6.35" y="-6.858" size="1.27" layer="27" ratio="10"/>
@@
 <attribute name="VALUE" x="-27.686" y="-296.4688" size="1.27" layer="27" ratio="10"/>
 </element>
-<element name="D7" library="diode" library_urn="urn:adsk.eagle:library:210" package="DO41-7.6" package3d_urn="urn:adsk.eagle:package:43421/1" value="1N5819-B" x="-25.4" y="-300.99" smashed="yes">
+<element name="D7" library="diode" library_urn="urn:adsk.eagle:library:210" package="DO41-7.6" package3d_urn="urn:adsk.eagle:package:43421/1" value="1N5819" x="-25.4" y="-300.99" smashed="yes">
 <attribute name="NAME" x="-27.432" y="-299.339" size="1.27" layer="25" ratio="10"/>
 <attribute name="VALUE" x="-27.432" y="-303.911" size="1.27" layer="27" ratio="10"/>
