File: projects/antenna-tuner/antenna-tuner.sch (EAGLE design)
At the start: 32 parts, among them J1 Power Jack, J2 RJ45, J3 RJ45, M1 SERVO, Q1 IRF5305, Q2 BC337, U1 Arduino Pro Mini

Commit message: Update copyright notice
Other:
- note added: "Copyright © 2018, Karim Hraibi Please visit: www.microfarad.de/magnetic-loop www.github.com/microfarad-de/antenna-tuner"
- note removed: "Copyright © 2018 Karim Hraibi Please visit: www.microfarad.de/magnetic-loop www.github.com/microfarad-de/antenna-tuner"
Changed lines of the file:
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@@
 <wire x1="-132.08" y1="-2.54" x2="-132.08" y2="114.3" width="0.1524" layer="95"/>
 <text x="-127" y="22.86" size="3.81" layer="95" align="top-left">Magnetic Loop Antenna Tuner</text>
-<text x="-127" y="15.24" size="2.1844" layer="95" align="top-left">Copyright © 2018 Karim Hraibi
+<text x="-127" y="15.24" size="2.1844" layer="95" align="top-left">Copyright © 2018, Karim Hraibi
 Please visit:
 www.microfarad.de/magnetic-loop
