File: projects/antenna-tuner/antenna-tuner.brd (EAGLE design)
At the start: 100 x 80 mm, 32 parts, among them J1 Power Jack, J2 RJ45, J3 RJ45, M1 SERVO, Q1 IRF5305, Q2 BC337, U1 Arduino Pro Mini

Commit message: Updated antenna tuner schematic
Parts:
- C3: value 10uF/25V tantal -> 10uF/25V Tantal
Changed lines of the file:
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@@
 <attribute name="VALUE" x="-56.4642" y="-69.2658" size="1.27" layer="27" ratio="10"/>
 </element>
-<element name="C3" library="rcl" library_urn="urn:adsk.eagle:library:334" package="E2,5-6" package3d_urn="urn:adsk.eagle:package:23349/1" value="10uF/25V tantal" x="-54.61" y="-74.93" smashed="yes">
+<element name="C3" library="rcl" library_urn="urn:adsk.eagle:library:334" package="E2,5-6" package3d_urn="urn:adsk.eagle:package:23349/1" value="10uF/25V Tantal" x="-54.61" y="-74.93" smashed="yes">
 <attribute name="NAME" x="-51.943" y="-73.406" size="1.27" layer="25" ratio="10"/>
 <attribute name="SPICEPREFIX" value="C" x="-54.61" y="-74.93" size="1.778" layer="27" display="off"/>
