File: projects/raspi-fan-control/fan-control.sch (EAGLE design)
At the start: 4 parts, among them J1 Raspberry Pi 40 Pin GPIO Head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, M1 Fan, T1 BC337

Commit message: Update copyright notice
Other:
- note added: "Copyright © 2018, Karim Hraibi Please visit: www.microfarad.de www.github.com/microfarad-de/nastia-server"
- note removed: "Please visit: www.microfarad.de www.githup.com/microfarad-de/nastia-server"
Changed lines of the file:
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@@
 <wire x1="93.98" y1="93.98" x2="93.98" y2="15.24" width="0.1524" layer="95"/>
 <wire x1="93.98" y1="15.24" x2="-5.08" y2="15.24" width="0.1524" layer="95"/>
-<text x="43.18" y="38.1" size="2.54" layer="95" align="top-left">Raspberry Pi Fan Control</text>
-<text x="43.18" y="33.02" size="1.778" layer="95" align="top-left">Please visit:
+<text x="43.18" y="40.64" size="2.54" layer="95" align="top-left">Raspberry Pi Fan Control</text>
+<text x="43.18" y="35.56" size="1.778" layer="95" align="top-left">Copyright © 2018, Karim Hraibi
+Please visit:
 www.microfarad.de
-www.githup.com/microfarad-de/nastia-server</text>
+www.github.com/microfarad-de/nastia-server</text>
 </plain>
 <instances>
