File: projects/li-charger/li-charger.sch (EAGLE design)
At the start: 24 parts, among them J1 Power Jack, Q1 IRF5305, Q2 BC547, U1 7805, U2 Arduino Pro Mini

Commit message: Update li-charger.sch
Parts:
- C4, C5: value 10µF Tantal -> 100nF
- R1: value 2K2 -> 470R
- R2: value 2K2 -> 220R
Other:
- note added: "Copyright © 2019, Karim Hraibi Please visit: www.microfarad.de/li-charger www.github.com/microfarad-de/li-charger"
- note removed: "Copyright © 2019, Karim Hraibi Please visit: www.microfarad.de www.github.com/microfarad-de/li-charger"
Changed lines of the file:
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@@
 <part name="P+1" library="supply1" library_urn="urn:adsk.eagle:library:371" deviceset="+12V" device="" value="+19.5V"/>
 <part name="C2" library="rcl" library_urn="urn:adsk.eagle:library:334" deviceset="C-EU" device="025-040X050" package3d_urn="urn:adsk.eagle:package:23634/1" value="330nF"/>
-<part name="R1" library="rcl" library_urn="urn:adsk.eagle:library:334" deviceset="R-EU_" device="0207/10" package3d_urn="urn:adsk.eagle:package:23491/2" value="2K2"/>
+<part name="R1" library="rcl" library_urn="urn:adsk.eagle:library:334" deviceset="R-EU_" device="0207/10" package3d_urn="urn:adsk.eagle:package:23491/2" value="470R"/>
 <part name="Q1" library="microfarad-de" deviceset="IRF5305" device=""/>
 <part name="J2" library="SparkFun-Connectors" library_urn="urn:adsk.eagle:library:513" deviceset="BANANA_CONN" device="" package3d_urn="urn:adsk.eagle:package:38018/1"/>
@@
 <part name="GND1" library="supply1" library_urn="urn:adsk.eagle:library:371" deviceset="0V" device=""/>
 <part name="Q2" library="transistor-npn" library_urn="urn:adsk.eagle:library:398" deviceset="BC547*" device="" package3d_urn="urn:adsk.eagle:package:28523/2"/>
-<part name="R2" library="rcl" library_urn="urn:adsk.eagle:library:334" deviceset="R-EU_" device="0207/10" package3d_urn="urn:adsk.eagle:package:23491/2" value="2K2"/>
+<part name="R2" library="rcl" library_urn="urn:adsk.eagle:library:334" deviceset="R-EU_" device="0207/10" package3d_urn="urn:adsk.eagle:package:23491/2" value="220R"/>
 <part name="D1" library="diode" library_urn="urn:adsk.eagle:library:210" deviceset="1N4004" device="" package3d_urn="urn:adsk.eagle:package:43336/1"/>
 <part name="U1" library="linear" library_urn="urn:adsk.eagle:library:262" deviceset="78*" device="TV" package3d_urn="urn:adsk.eagle:package:16417/1" technology="05" value="7805"/>
 <part name="C1" library="rcl" library_urn="urn:adsk.eagle:library:334" deviceset="CPOL-EU" device="E2.5-5" package3d_urn="urn:adsk.eagle:package:23344/1" value="100µF"/>
-<part name="C4" library="rcl" library_urn="urn:adsk.eagle:library:334" deviceset="CPOL-EU" device="E2.5-5" package3d_urn="urn:adsk.eagle:package:23344/1" value="10µF Tantal"/>
-<part name="C5" library="rcl" library_urn="urn:adsk.eagle:library:334" deviceset="CPOL-EU" device="E2.5-5" package3d_urn="urn:adsk.eagle:package:23344/1" value="10µF Tantal"/>
+<part name="C4" library="rcl" library_urn="urn:adsk.eagle:library:334" deviceset="CPOL-EU" device="E2.5-5" package3d_urn="urn:adsk.eagle:package:23344/1" value="100nF"/>
+<part name="C5" library="rcl" library_urn="urn:adsk.eagle:library:334" deviceset="CPOL-EU" device="E2.5-5" package3d_urn="urn:adsk.eagle:package:23344/1" value="100nF"/>
 <part name="R9" library="rcl" library_urn="urn:adsk.eagle:library:334" deviceset="R-EU_" device="0617/22" package3d_urn="urn:adsk.eagle:package:23577/1" value="1R/3W"/>
 <part name="D2" library="diode" library_urn="urn:adsk.eagle:library:210" deviceset="BY251" device="" package3d_urn="urn:adsk.eagle:package:43365/1" value="BY255"/>
@@
 <text x="20.32" y="-7.62" size="2.1844" layer="95" align="top-left">Copyright © 2019, Karim Hraibi
 Please visit:
-www.microfarad.de
+www.microfarad.de/li-charger
 www.github.com/microfarad-de/li-charger</text>
 <text x="56.642" y="13.97" size="1.778" layer="95" rot="R90">Shunt</text>
@@
 </instance>
 <instance part="R7" gate="G$1" x="12.7" y="17.78" smashed="yes" rot="R90">
-<attribute name="NAME" x="11.2014" y="13.97" size="1.778" layer="95" rot="R90"/>
+<attribute name="NAME" x="10.9474" y="14.224" size="1.778" layer="95" rot="R90"/>
 <attribute name="VALUE" x="16.002" y="13.97" size="1.778" layer="96" rot="R90"/>
 </instance>
@@
 </instance>
 <instance part="C4" gate="G$1" x="5.08" y="17.78" smashed="yes">
-<attribute name="NAME" x="7.493" y="18.2626" size="1.778" layer="95" rot="R90"/>
-<attribute name="VALUE" x="2.921" y="7.8486" size="1.778" layer="96" rot="R90"/>
+<attribute name="NAME" x="2.667" y="11.4046" size="1.778" layer="95" rot="R90"/>
+<attribute name="VALUE" x="2.667" y="15.9766" size="1.778" layer="96" rot="R90"/>
 </instance>
 <instance part="C5" gate="G$1" x="22.86" y="17.78" smashed="yes">
-<attribute name="NAME" x="25.273" y="18.2626" size="1.778" layer="95" rot="R90"/>
-<attribute name="VALUE" x="20.701" y="7.8486" size="1.778" layer="96" rot="R90"/>
+<attribute name="NAME" x="20.701" y="11.4046" size="1.778" layer="95" rot="R90"/>
+<attribute name="VALUE" x="20.447" y="15.9766" size="1.778" layer="96" rot="R90"/>
 </instance>
 <instance part="R9" gate="G$1" x="63.5" y="17.78" smashed="yes" rot="R90">

Commit message: Updated li-charger
Parts:
- C4, C5: device rcl:CPOL-EUE2.5-5 -> rcl:C-EU025-040X050
Connections:
- net 0V: now also C4.2, C5.2; no longer C4.-, C5.-
- net N$10: now also C4.1; no longer C4.+
- net N$13: now also C5.1; no longer C5.+
Changed lines of the file:
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@@
 <part name="U1" library="linear" library_urn="urn:adsk.eagle:library:262" deviceset="78*" device="TV" package3d_urn="urn:adsk.eagle:package:16417/1" technology="05" value="7805"/>
 <part name="C1" library="rcl" library_urn="urn:adsk.eagle:library:334" deviceset="CPOL-EU" device="E2.5-5" package3d_urn="urn:adsk.eagle:package:23344/1" value="100µF"/>
-<part name="C4" library="rcl" library_urn="urn:adsk.eagle:library:334" deviceset="CPOL-EU" device="E2.5-5" package3d_urn="urn:adsk.eagle:package:23344/1" value="100nF"/>
-<part name="C5" library="rcl" library_urn="urn:adsk.eagle:library:334" deviceset="CPOL-EU" device="E2.5-5" package3d_urn="urn:adsk.eagle:package:23344/1" value="100nF"/>
 <part name="R9" library="rcl" library_urn="urn:adsk.eagle:library:334" deviceset="R-EU_" device="0617/22" package3d_urn="urn:adsk.eagle:package:23577/1" value="1R/3W"/>
 <part name="D2" library="diode" library_urn="urn:adsk.eagle:library:210" deviceset="BY251" device="" package3d_urn="urn:adsk.eagle:package:43365/1" value="BY255"/>
+<part name="C4" library="rcl" library_urn="urn:adsk.eagle:library:334" deviceset="C-EU" device="025-040X050" package3d_urn="urn:adsk.eagle:package:23634/1" value="100nF"/>
+<part name="C5" library="rcl" library_urn="urn:adsk.eagle:library:334" deviceset="C-EU" device="025-040X050" package3d_urn="urn:adsk.eagle:package:23634/1" value="100nF"/>
 </parts>
 <sheets>
@@
 <attribute name="VALUE" x="-21.209" y="66.2686" size="1.778" layer="96" rot="R90"/>
 </instance>
-<instance part="C4" gate="G$1" x="5.08" y="17.78" smashed="yes">
-<attribute name="NAME" x="2.667" y="11.4046" size="1.778" layer="95" rot="R90"/>
-<attribute name="VALUE" x="2.667" y="15.9766" size="1.778" layer="96" rot="R90"/>
-</instance>
-<instance part="C5" gate="G$1" x="22.86" y="17.78" smashed="yes">
-<attribute name="NAME" x="20.701" y="11.4046" size="1.778" layer="95" rot="R90"/>
-<attribute name="VALUE" x="20.447" y="15.9766" size="1.778" layer="96" rot="R90"/>
-</instance>
 <instance part="R9" gate="G$1" x="63.5" y="17.78" smashed="yes" rot="R90">
 <attribute name="NAME" x="63.0174" y="20.828" size="1.778" layer="95" rot="R90"/>
@@
 <attribute name="NAME" x="58.9026" y="60.96" size="1.778" layer="95" rot="R270"/>
 <attribute name="VALUE" x="56.1086" y="60.96" size="1.778" layer="96" rot="R270"/>
+</instance>
+<instance part="C4" gate="G$1" x="5.08" y="17.78" smashed="yes">
+<attribute name="NAME" x="4.318" y="18.161" size="1.778" layer="95" rot="R90"/>
+<attribute name="VALUE" x="4.318" y="8.255" size="1.778" layer="96" rot="R90"/>
+</instance>
+<instance part="C5" gate="G$1" x="22.86" y="17.78" smashed="yes">
+<attribute name="NAME" x="22.098" y="18.161" size="1.778" layer="95" rot="R90"/>
+<attribute name="VALUE" x="22.098" y="8.255" size="1.778" layer="96" rot="R90"/>
 </instance>
 </instances>
@@
 <wire x1="22.86" y1="5.08" x2="22.86" y2="12.7" width="0.1524" layer="91"/>
 <wire x1="12.7" y1="2.54" x2="12.7" y2="5.08" width="0.1524" layer="91"/>
-<pinref part="C4" gate="G$1" pin="-"/>
-<pinref part="C5" gate="G$1" pin="-"/>
+<pinref part="C4" gate="G$1" pin="2"/>
+<pinref part="C5" gate="G$1" pin="2"/>
 </segment>
 <segment>
@@
 <wire x1="12.7" y1="22.86" x2="12.7" y2="30.48" width="0.1524" layer="91"/>
 <junction x="12.7" y="30.48"/>
-<pinref part="C4" gate="G$1" pin="+"/>
+<pinref part="C4" gate="G$1" pin="1"/>
 </segment>
 </net>
@@
 <wire x1="22.86" y1="20.32" x2="22.86" y2="27.94" width="0.1524" layer="91"/>
 <junction x="22.86" y="27.94"/>
-<pinref part="C5" gate="G$1" pin="+"/>
-</segment>
-</net>
+<pinref part="C5" gate="G$1" pin="1"/>
+</segment>
+</net>
